File: extension_mb1136/extension_mb1136.kicad_pcb (KiCad board)
At the start: 2 copper layers, 26 parts, among them CN1 Conn_02x19_Odd_Even, CN2 Conn_02x19_Odd_Even, CN3 Conn_01x08, CN4 Conn_01x06, CN5 Conn_01x08, CN6 Conn_01x10, J1 Conn_01x03, J2 Conn_01x03, Q1 S9013, U1 STMPS2151MTR, U2 USBLC6-2

Commit message: add poligons project
Parts:
- moved R7 37.1 mm to (53.8, 61.7), turned to 90 degrees
- moved R1 36.6 mm to (47.6, 66.0), turned to 90 degrees
- moved LD1 35.5 mm to (47.8, 61.7), turned to 270 degrees
- moved R2 32.6 mm to (50.8, 66.0), turned to 90 degrees
- moved R8 31.6 mm to (43.9, 78.9), turned to 270 degrees
- moved R4 29.9 mm to (47.5, 69.8), turned to 270 degrees
- moved R6 29.3 mm to (53.8, 69.0), turned to 270 degrees
- moved CNUSB_1 28.8 mm to (40.6, 99.1)
- moved C1 26.7 mm to (37.6, 80.8), turned to 90 degrees
- moved R9 26.6 mm to (75.8, 68.8), turned to 180 degrees
- moved R5 25.8 mm to (53.8, 65.3), turned to 90 degrees
- moved U2 24.7 mm to (56.1, 82.0)
- moved CNUSB_2 23.6 mm to (52.6, 89.4)
- moved R3 22.1 mm to (70.1, 67.3), turned to 270 degrees
- moved D1 20.2 mm to (46.5, 98.9), turned to 270 degrees
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
Commit message: add connector, develop pcb
Parts:
- added CNUSB_1: USB_B, Connector_USB:USB_B_OST_USB-B1HSxx_Horizontal, F.Cu at (72.4, 88.9)
- moved C1 24.7 mm to (46.2, 57.7)
- moved R6 24.3 mm to (43.4, 54.6), turned to 90 degrees
- moved Q1 22.3 mm to (38.9, 58.4), turned to 270 degrees
- moved LD1 18.8 mm to (38.9, 63.5), turned to 270 degrees
- moved R4 18.1 mm to (52.3, 64.0), turned to 180 degrees
- moved U2 16.7 mm to (47.6, 64.1), turned to 90 degrees
- moved R5 15.0 mm to (43.4, 58.2), turned to 90 degrees
- moved J2 12.5 mm to (61.5, 59.6), turned to 180 degrees
- moved D1 10.8 mm to (36.8, 94.0), turned to 180 degrees
- moved J1 10.0 mm to (57.0, 59.6), turned to 180 degrees
- moved R8 9.12 mm to (41.9, 68.1), turned to 0 degrees
- moved R7 9.00 mm to (38.9, 67.3), turned to 90 degrees
- moved R2 7.61 mm to (50.5, 58.4), turned to 0 degrees
- moved R3 6.27 mm to (50.5, 56.4), turned to 180 degrees
- moved LD2 5.88 mm to (42.0, 63.1), turned to 180 degrees
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- renumbered CNUSB_1 to CNUSB_2, CNUSB_2 to CNUSB_3, LD2 to LD1, LD1 to LD2, R9 to R1, R5 to R2, R7 to R3, R3 to R4, R6 to R5, R8 to R6, R4 to R7, R2 to R8, R1 to R9, U2 to U1, U1 to U2
Routing:
- net PC8: track 0.00 -> 39.4 mm
- net PC9: track 0.00 -> 29.3 mm
- net +5V: track 0.00 -> 25.0 mm
- net PA9: track 0.00 -> 18.5 mm
- net VBUS_DET: track 0.00 -> 17.1 mm, vias 0 -> 2
- net USB_OWER_CURRENT: track 0.00 -> 13.7 mm
- net USB_POWER_SWITCH_ON: track 0.00 -> 13.1 mm
- net +3V3: track 0.00 -> 9.74 mm
- net PA7: track 0.00 -> 5.71 mm
- net PA5: track 0.00 -> 5.71 mm
- net PB9: track 0.00 -> 5.71 mm
- net PB8: track 0.00 -> 5.71 mm
- net GND: track 0.00 -> 5.71 mm
- net AVDD: track 0.00 -> 5.71 mm
- net PC7: track 0.00 -> 5.71 mm
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Other:
- board outline added: 70 x 57.5 mm

Commit message: update pcb
Parts:
- moved R1 26.3 mm to (54.4, 53.6), turned to 270 degrees
- moved D1 22.1 mm to (58.7, 90.9), turned to 0 degrees
- moved CNUSB_2 17.3 mm to (57.9, 100.6)
- moved CNUSB_3 9.65 mm to (41.1, 91.4)
- moved LD2 5.21 mm to (42.2, 68.3)
- moved R8 5.09 mm to (42.2, 63.0)
Routing:
- net PA9: track 18.5 -> 116.6 mm, vias 0 -> 2
- net PB12: track 0.00 -> 91.7 mm, vias 0 -> 2
- net PA11: track 0.00 -> 91.5 mm, vias 0 -> 1
- net Net-(CNUSB_1-Pad2): track 0.00 -> 54.4 mm, vias 0 -> 2
- net Net-(CNUSB_1-Pad3): track 0.00 -> 51.2 mm, vias 0 -> 2
- net USB_OWER_CURRENT: track 13.7 -> 28.0 mm, vias 0 -> 1
- net +3V3: track 9.74 -> 18.5 mm
- net USB_DISCONNECT: track 0.00 -> 2.68 mm
- net VBUS_DET: track 17.1 -> 18.5 mm

Commit message: update pcb
Parts:
- removed the CNUSB_1 at (72.4, 88.9)
- added CNUSB_3: USB_BP, Connector_USB:USB_B_OST_USB-B1HSxx_Horizontal, F.Cu at (44.7, 88.9)
- added D2: D, Diode_SMD:D_0805_2012Metric, F.Cu at (66.2, 65.3)
- added SW1: USB_SEL, Connector_PinSocket_2.54mm:PinSocket_2x03_P2.54mm_Vertical, F.Cu at (38.6, 77.0)
- added SW2: USB_SEL, Connector_PinSocket_2.54mm:PinSocket_2x03_P2.54mm_Vertical, F.Cu at (45.0, 82.0)
- moved CNUSB_2 26.7 mm to (67.8, 91.4)
- moved U2 10.2 mm to (55.1, 71.9)
- moved D1 10.1 mm to (63.5, 99.8)
- moved R3 5.44 mm to (57.8, 64.0), turned to 0 degrees
- renumbered CNUSB_2 to CNUSB_1, CNUSB_3 to CNUSB_2, LD2 to LD1, LD1 to LD2, R9 to R1, R8 to R2, R4 to R3, R7 to R4, R2 to R5, R5 to R6, R3 to R7, R6 to R8, R1 to R9, U2 to U1, U1 to U2
Connections:
- CNUSB_2 pad 2: Net-(CNUSB_1-Pad2) -> Net-(CNUSB_2-Pad2)
- CNUSB_2 pad 3: Net-(CNUSB_1-Pad3) -> Net-(CNUSB_2-Pad3)
- U2 pad 4: Net-(CNUSB_1-Pad2) -> Net-(SW2-Pad3)
- U2 pad 6: Net-(CNUSB_1-Pad3) -> Net-(SW1-Pad3)
Routing:
- net PA9: track 116.6 -> 20.2 mm, vias 2 -> 1
- net Net-(CNUSB_1-Pad2): track 54.4 -> 0.00 mm, vias 2 -> 0
- net Net-(CNUSB_1-Pad3): track 51.2 -> 0.00 mm, vias 2 -> 0
- net PA11: track 91.5 -> 80.6 mm
- net PB12: track 91.7 -> 81.3 mm
- net PA5: track 5.71 -> 4.05 mm
- net GND: track 5.71 -> 4.05 mm
- net Net-(CNUSB_3-Pad1): track 0.00 -> 1.27 mm

Commit message: update pcb
Parts:
- added D3: D, Diode_SMD:D_0805_2012Metric_Pad1.15x1.40mm_HandSolder, F.Cu at (42.8, 72.6)
- D2: footprint Diode_SMD:D_0805_2012Metric -> Diode_SMD:D_0805_2012Metric_Pad1.15x1.40mm_HandSolder
- moved D2 22.6 mm to (44.8, 72.6), turned to 270 degrees
- moved SW1 20.3 mm to (58.0, 83.0), turned to 180 degrees
- moved D1 7.50 mm to (59.3, 93.6)
- moved SW2 5.10 mm to (50.0, 83.0), turned to 180 degrees
- moved U2 1.66 mm to (55.0, 70.2)
Connections:
- D2 pad 1: +5V -> +5VD
- U1 pad 2: +5V -> +5VD
- U1 pad 3: +5V -> +5VD
Routing:
- net PA9: track 20.2 -> 103.2 mm, vias 1 -> 4
- net Net-(CNUSB_2-Pad2): track 0.00 -> 39.8 mm, vias 0 -> 1
- net PB10: track 5.08 -> 38.7 mm, vias 0 -> 1
- net Net-(CNUSB_2-Pad3): track 0.00 -> 31.7 mm, vias 0 -> 1
- net Net-(CNUSB_3-Pad3): track 0.00 -> 26.4 mm, vias 0 -> 1
- net Net-(CNUSB_1-Pad3): track 0.00 -> 22.3 mm
- net Net-(CNUSB_1-Pad2): track 0.00 -> 21.8 mm
- net Net-(SW2-Pad3): track 0.00 -> 15.0 mm
- net Net-(CNUSB_3-Pad1): track 1.27 -> 15.3 mm
- net Net-(CNUSB_3-Pad2): track 0.00 -> 13.7 mm, vias 0 -> 1
- net +5V: track 25.0 -> 14.8 mm
- net Net-(SW1-Pad3): track 0.00 -> 9.73 mm
- net +5VD: track 0.00 -> 9.09 mm
- net PB12: track 81.3 -> 79.2 mm
- net PA11: track 80.6 -> 78.6 mm

Commit message: update pcb
Routing:
- added copper zone on F.Cu, net GND
Changed lines of the file:
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@@
     (trace_clearance 0.2)
     (zone_clearance 0.508)
-    (zone_45_only no)
+    (zone_45_only yes)
     (trace_min 0.2)
     (via_size 0.8)
@@
   (segment (start 44.778 71.046) (end 46.99 68.834) (width 0.5) (layer F.Cu) (net 94))
   (segment (start 44.778 71.61) (end 44.778 71.046) (width 0.25) (layer F.Cu) (net 94))
+  (zone (net 2) (net_name GND) (layer F.Cu) (hatch edge 0.508)
+    (priority 100)
+    (connect_pads (clearance 0.508))
+    (min_thickness 0.254)
+    (fill yes (arc_segments 32) (thermal_gap 0.508) (thermal_bridge_width 0.508))
+    (polygon
+      (pts
+        (xy 40.767 74.803) (xy 43.561 76.073) (xy 43.815 81.407) (xy 39.497 81.534) (xy 39.37 92.075)
+        (xy 43.053 93.218) (xy 43.688 90.297) (xy 47.371 90.297) (xy 47.498 86.487) (xy 55.118 86.614)
+        (xy 56.134 97.409) (xy 56.134 100.711) (xy 59.436 100.711) (xy 60.833 92.329) (xy 66.04 92.329)
+        (xy 67.437 94.361) (xy 74.803 94.361) (xy 76.962 92.075) (xy 79.502 92.075) (xy 79.629 102.997)
+        (xy 34.798 103.251) (xy 34.9885 92.1385) (xy 34.925 79.883) (xy 26.67 80.01) (xy 26.67 77.597)
+        (xy 23.622 77.597) (xy 23.622 75.057) (xy 35.56 74.93)
+      )
+    )
+  )
 )

Commit message: update pcb
Routing:
- net GND: track 4.05 -> 16.5 mm, vias 0 -> 214
- net PA5: track 4.05 -> 5.71 mm
- net PA9: track 103.2 -> 102.3 mm
- net PB12: track 79.2 -> 79.4 mm, vias 2 -> 3
- added copper zone on B.Cu, net GND
